Commit message: new urdf file for 3 DOF arm

File: PassThrough/basic_arm.urdf (robot description, URDF)
Before this commit: robot myfirst, 4 links, 3 joints
Links:
- removed link bottom_arm
- removed link middle_arm
- removed link top_arm
- added link link1; collision box size=0.1 0.1 1; visual box size=0.1 0.1 1
- added link link2; collision box size=0.1 0.1 1; visual box size=0.1 0.1 1
- added link link3; collision box size=0.1 0.1 1; visual box size=0.1 0.1 1
Joints:
- removed joint base_to_bottom
- removed joint bottom_to_middle
- removed joint middle_to_top
- added joint base_link1: type continuous, parent base, child link1, origin xyz=0 0 0.1, axis 0 0 1
- added joint link1_link2: type continuous, parent link1, child link2, origin xyz=0 0 1, axis 0 1 0
- added joint link2_link3: type continuous, parent link2, child link3, origin xyz=0 0 1, axis 0 1 0
