Commit message: made 3DOF simulation, ML based method still faster than sampling, ML has decent accuracy (97%), plotting them in 3D

File: 3DOF/basic_arm.urdf (robot description, URDF)
Before this commit: robot myfirst, 4 links, 3 joints
Links:
- link base: mass None -> 10
- link link_1: mass None -> 10
- link link_2: mass None -> 10
- link link_3: mass None -> 10
Joints:
- joint base_link1: child link1 -> link_1
- joint link1_link2: child link2 -> link_2; parent link1 -> link_1
- joint link2_link3: child link3 -> link_3; parent link2 -> link_2
